Commit message: Correct WR141E geometry and four-panel Underbot R10 enclosure

File: underbot_description/urdf/arm.xacro (robot description, xacro)
@@ -403,5 +403,5 @@
       <parent link="base_link" />
       <child link="left_arm_base" />
-      <origin xyz="-0.07 0.108 0.545" rpy="0 -1.57079632679 -1.57079632679" />
+      <origin xyz="-0.14 0.108 0.545" rpy="0 -1.57079632679 -1.57079632679" />
       <axis xyz="0 0 1" />
       <limit effort="1" velocity="1" lower="-0.785398163397" upper="0.785398163397" />
@@ -460,5 +460,5 @@
       <parent link="base_link" />
       <child link="right_arm_base" />
-      <origin xyz="-0.07 -0.108 0.545" rpy="0 -1.57079632679 1.57079632679" />
+      <origin xyz="-0.14 -0.108 0.545" rpy="0 -1.57079632679 1.57079632679" />
       <axis xyz="0 0 -1" />
       <limit effort="1" velocity="1" lower="-0.785398163397" upper="0.785398163397" />

File: underbot_description/urdf/base.xacro (robot description, xacro)
@@ -4,7 +4,7 @@
     <link name="base_link">
       <inertial>
-        <origin xyz="-0.0598350198234 5.40649302867e-05 0.274770185411" rpy="0 0 0" />
-        <mass value="14.8710078" />
-        <inertia ixx="0.627048766532" ixy="8.172644062e-06" ixz="0.0129279632493" iyy="0.700954782211" iyz="-5.60167709298e-05" izz="0.256652248656" />
+        <origin xyz="-0.0675738134449 5.43711724368e-05 0.264312407779" rpy="0 0 0" />
+        <mass value="14.7872478" />
+        <inertia ixx="0.692717397506" ixy="5.82306539903e-05" ixz="0.170292249867" iyy="0.856120402596" iyz="-6.44248241453e-05" izz="0.411854129182" />
       </inertial>
       <visual name="base_link_visual_0">
@@ -14,5 +14,5 @@
         </geometry>
         <material name="matte_black">
-          <color rgba="0.045 0.05 0.055 1" />
+          <color rgba="0.008 0.009 0.011 1" />
         </material>
       </visual>
@@ -38,4 +38,13 @@
         <origin xyz="0 0 0" rpy="0 0 0" />
         <geometry>
+          <mesh filename="package://underbot_description/meshes/base_link_aluminium.stl" scale="1 1 1" />
+        </geometry>
+        <material name="aluminium">
+          <color rgba="0.62 0.68 0.72 1" />
+        </material>
+      </visual>
+      <visual name="base_link_visual_4">
+        <origin xyz="0 0 0" rpy="0 0 0" />
+        <geometry>
           <mesh filename="package://underbot_description/meshes/base_link_control_red.stl" scale="1 1 1" />
         </geometry>
@@ -44,23 +53,5 @@
         </material>
       </visual>
-      <visual name="base_link_visual_4">
-        <origin xyz="0 0 0" rpy="0 0 0" />
-        <geometry>
-          <mesh filename="package://underbot_description/meshes/base_link_aluminium.stl" scale="1 1 1" />
-        </geometry>
-        <material name="aluminium">
-          <color rgba="0.62 0.68 0.72 1" />
-        </material>
-      </visual>
       <visual name="base_link_visual_5">
-        <origin xyz="0 0 0" rpy="0 0 0" />
-        <geometry>
-          <mesh filename="package://underbot_description/meshes/base_link_polycarbonate.stl" scale="1 1 1" />
-        </geometry>
-        <material name="polycarbonate">
-          <color rgba="0.38 0.55 0.6 0.5" />
-        </material>
-      </visual>
-      <visual name="base_link_visual_6">
         <origin xyz="0 0 0" rpy="0 0 0" />
         <geometry>
@@ -71,60 +62,63 @@
         </material>
       </visual>
+      <visual name="base_link_visual_6">
+        <origin xyz="0 0 0" rpy="0 0 0" />
+        <geometry>
+          <mesh filename="package://underbot_description/meshes/base_link_polycarbonate.stl" scale="1 1 1" />
+        </geometry>
+        <material name="polycarbonate">
+          <color rgba="0.94 0.975 0.99 0.16" />
+        </material>
+      </visual>
       <collision name="base_link_rear_chassis">
-        <origin xyz="-0.0675 0 0.1225" rpy="0 0 0" />
-        <geometry>
-          <box size="0.375 0.296 0.115" />
+        <origin xyz="-0.09 0 0.1175" rpy="0 0 0" />
+        <geometry>
+          <box size="0.37 0.28 0.105" />
         </geometry>
       </collision>
       <collision name="base_link_nose_side_-1">
-        <origin xyz="0.2 -0.11 0.115" rpy="0 0 0" />
-        <geometry>
-          <box size="0.15 0.08 0.09" />
+        <origin xyz="0.155 -0.133 0.105" rpy="0 0 0" />
+        <geometry>
+          <box size="0.15 0.065 0.07" />
         </geometry>
       </collision>
       <collision name="base_link_nose_side_1">
-        <origin xyz="0.2 0.11 0.115" rpy="0 0 0" />
-        <geometry>
-          <box size="0.15 0.08 0.09" />
+        <origin xyz="0.155 0.133 0.105" rpy="0 0 0" />
+        <geometry>
+          <box size="0.15 0.065 0.07" />
         </geometry>
       </collision>
       <collision name="base_link_nose_upper">
-        <origin xyz="0.194 0 0.174" rpy="0 0 0" />
-        <geometry>
-          <box size="0.17 0.29 0.028" />
-        </geometry>
-      </collision>
-      <collision name="base_link_front_grille">
-        <origin xyz="0.2775 0 0.12" rpy="0 0 0" />
-        <geometry>
-          <box size="0.003 0.29 0.07" />
+        <origin xyz="0.16 0 0.143" rpy="0 0 0" />
+        <geometry>
+          <box size="0.18 0.28 0.035" />
         </geometry>
       </collision>
       <collision name="base_link_chassis_adapter">
-        <origin xyz="-0.07 0 0.202" rpy="0 0 0" />
+        <origin xyz="-0.14 0 0.202" rpy="0 0 0" />
         <geometry>
           <box size="0.2 0.2 0.006" />
         </geometry>
       </collision>
-      <collision name="base_link_post_-0.16000000000000003_-0.09000000000000001">
-        <origin xyz="-0.16 -0.09 0.455" rpy="0 0 0" />
+      <collision name="base_link_post_-0.23000000000000004_-0.09000000000000001">
+        <origin xyz="-0.23 -0.09 0.455" rpy="0 0 0" />
         <geometry>
           <box size="0.02 0.02 0.5" />
         </geometry>
       </collision>
-      <collision name="base_link_post_-0.16000000000000003_0.09000000000000001">
-        <origin xyz="-0.16 0.09 0.455" rpy="0 0 0" />
+      <collision name="base_link_post_-0.23000000000000004_0.09000000000000001">
+        <origin xyz="-0.23 0.09 0.455" rpy="0 0 0" />
         <geometry>
           <box size="0.02 0.02 0.5" />
         </geometry>
       </collision>
-      <collision name="base_link_post_0.020000000000000004_-0.09000000000000001">
-        <origin xyz="0.02 -0.09 0.455" rpy="0 0 0" />
+      <collision name="base_link_post_-0.05_-0.09000000000000001">
+        <origin xyz="-0.05 -0.09 0.455" rpy="0 0 0" />
         <geometry>
           <box size="0.02 0.02 0.5" />
         </geometry>
       </collision>
-      <collision name="base_link_post_0.020000000000000004_0.09000000000000001">
-        <origin xyz="0.02 0.09 0.455" rpy="0 0 0" />
+      <collision name="base_link_post_-0.05_0.09000000000000001">
+        <origin xyz="-0.05 0.09 0.455" rpy="0 0 0" />
         <geometry>
           <box size="0.02 0.02 0.5" />
@@ -132,5 +126,5 @@
       </collision>
       <collision name="base_link_rail_x_0_-1">
-        <origin xyz="-0.07 -0.09 0.215" rpy="0 0 0" />
+        <origin xyz="-0.14 -0.09 0.215" rpy="0 0 0" />
         <geometry>
           <box size="0.16 0.02 0.02" />
@@ -138,5 +132,5 @@
       </collision>
       <collision name="base_link_rail_y_0_-1">
-        <origin xyz="-0.16 0 0.215" rpy="0 0 0" />
+        <origin xyz="-0.23 0 0.215" rpy="0 0 0" />
         <geometry>
           <box size="0.02 0.16 0.02" />
@@ -144,5 +138,5 @@
       </collision>
       <collision name="base_link_rail_x_0_1">
-        <origin xyz="-0.07 0.09 0.215" rpy="0 0 0" />
+        <origin xyz="-0.14 0.09 0.215" rpy="0 0 0" />
         <geometry>
           <box size="0.16 0.02 0.02" />
@@ -150,5 +144,5 @@
       </collision>
       <collision name="base_link_rail_y_0_1">
-        <origin xyz="0.02 0 0.215" rpy="0 0 0" />
+        <origin xyz="-0.05 0 0.215" rpy="0 0 0" />
         <geometry>
           <box size="0.02 0.16 0.02" />
@@ -156,5 +150,5 @@
       </collision>
       <collision name="base_link_floor_0_center">
-        <origin xyz="-0.07 0 0.2265" rpy="0 0 0" />
+        <origin xyz="-0.14 0 0.2265" rpy="0 0 0" />
         <geometry>
           <box size="0.16 0.2 0.003" />
@@ -162,5 +156,5 @@
       </collision>
       <collision name="base_link_floor_0_end_-1">
-        <origin xyz="-0.16 0 0.2265" rpy="0 0 0" />
+        <origin xyz="-0.23 0 0.2265" rpy="0 0 0" />
         <geometry>
           <box size="0.02 0.16 0.003" />
@@ -168,5 +162,5 @@
       </collision>
       <collision name="base_link_floor_0_end_1">
-        <origin xyz="0.02 0 0.2265" rpy="0 0 0" />
+        <origin xyz="-0.05 0 0.2265" rpy="0 0 0" />
         <geometry>
           <box size="0.02 0.16 0.003" />
@@ -174,5 +168,5 @@
       </collision>
       <collision name="base_link_rail_x_1_-1">
-        <origin xyz="-0.07 -0.09 0.49" rpy="0 0 0" />
+        <origin xyz="-0.14 -0.09 0.49" rpy="0 0 0" />
         <geometry>
           <box size="0.16 0.02 0.02" />
@@ -180,5 +174,5 @@
       </collision>
       <collision name="base_link_rail_y_1_-1">
-        <origin xyz="-0.16 0 0.49" rpy="0 0 0" />
+        <origin xyz="-0.23 0 0.49" rpy="0 0 0" />
         <geometry>
           <box size="0.02 0.16 0.02" />
@@ -186,5 +180,5 @@
       </collision>
       <collision name="base_link_rail_x_1_1">
-        <origin xyz="-0.07 0.09 0.49" rpy="0 0 0" />
+        <origin xyz="-0.14 0.09 0.49" rpy="0 0 0" />
         <geometry>
           <box size="0.16 0.02 0.02" />
@@ -192,5 +186,5 @@
       </collision>
       <collision name="base_link_rail_y_1_1">
-        <origin xyz="0.02 0 0.49" rpy="0 0 0" />
+        <origin xyz="-0.05 0 0.49" rpy="0 0 0" />
         <geometry>
           <box size="0.02 0.16 0.02" />
@@ -198,5 +192,5 @@
       </collision>
       <collision name="base_link_floor_1_center">
-        <origin xyz="-0.07 0 0.5015" rpy="0 0 0" />
+        <origin xyz="-0.14 0 0.5015" rpy="0 0 0" />
         <geometry>
           <box size="0.16 0.2 0.003" />
@@ -204,5 +198,5 @@
       </collision>
       <collision name="base_link_floor_1_end_-1">
-        <origin xyz="-0.16 0 0.5015" rpy="0 0 0" />
+        <origin xyz="-0.23 0 0.5015" rpy="0 0 0" />
         <geometry>
           <box size="0.02 0.16 0.003" />
@@ -210,5 +204,5 @@
       </collision>
       <collision name="base_link_floor_1_end_1">
-        <origin xyz="0.02 0 0.5015" rpy="0 0 0" />
+        <origin xyz="-0.05 0 0.5015" rpy="0 0 0" />
         <geometry>
           <box size="0.02 0.16 0.003" />
@@ -216,5 +210,5 @@
       </collision>
       <collision name="base_link_rail_x_2_-1">
-        <origin xyz="-0.07 -0.09 0.565" rpy="0 0 0" />
+        <origin xyz="-0.14 -0.09 0.565" rpy="0 0 0" />
         <geometry>
           <box size="0.16 0.02 0.02" />
@@ -222,5 +216,5 @@
       </collision>
       <collision name="base_link_rail_y_2_-1">
-        <origin xyz="-0.16 0 0.565" rpy="0 0 0" />
+        <origin xyz="-0.23 0 0.565" rpy="0 0 0" />
         <geometry>
           <box size="0.02 0.16 0.02" />
@@ -228,5 +222,5 @@
       </collision>
       <collision name="base_link_rail_x_2_1">
-        <origin xyz="-0.07 0.09 0.565" rpy="0 0 0" />
+        <origin xyz="-0.14 0.09 0.565" rpy="0 0 0" />
         <geometry>
           <box size="0.16 0.02 0.02" />
@@ -234,5 +228,5 @@
       </collision>
       <collision name="base_link_rail_y_2_1">
-        <origin xyz="0.02 0 0.565" rpy="0 0 0" />
+        <origin xyz="-0.05 0 0.565" rpy="0 0 0" />
         <geometry>
           <box size="0.02 0.16 0.02" />
@@ -240,5 +234,5 @@
       </collision>
       <collision name="base_link_floor_2_center">
-        <origin xyz="-0.07 0 0.5765" rpy="0 0 0" />
+        <origin xyz="-0.14 0 0.5765" rpy="0 0 0" />
         <geometry>
           <box size="0.16 0.2 0.003" />
@@ -246,5 +240,5 @@
       </collision>
       <collision name="base_link_floor_2_end_-1">
-        <origin xyz="-0.16 0 0.5765" rpy="0 0 0" />
+        <origin xyz="-0.23 0 0.5765" rpy="0 0 0" />
         <geometry>
           <box size="0.02 0.16 0.003" />
@@ -252,5 +246,5 @@
       </collision>
       <collision name="base_link_floor_2_end_1">
-        <origin xyz="0.02 0 0.5765" rpy="0 0 0" />
+        <origin xyz="-0.05 0 0.5765" rpy="0 0 0" />
         <geometry>
           <box size="0.02 0.16 0.003" />
@@ -258,5 +252,5 @@
       </collision>
       <collision name="base_link_rail_x_3_-1">
-        <origin xyz="-0.07 -0.09 0.695" rpy="0 0 0" />
+        <origin xyz="-0.14 -0.09 0.695" rpy="0 0 0" />
         <geometry>
           <box size="0.16 0.02 0.02" />
@@ -264,5 +258,5 @@
       </collision>
       <collision name="base_link_rail_y_3_-1">
-        <origin xyz="-0.16 0 0.695" rpy="0 0 0" />
+        <origin xyz="-0.23 0 0.695" rpy="0 0 0" />
         <geometry>
           <box size="0.02 0.16 0.02" />
@@ -270,5 +264,5 @@
       </collision>
       <collision name="base_link_rail_x_3_1">
-        <origin xyz="-0.07 0.09 0.695" rpy="0 0 0" />
+        <origin xyz="-0.14 0.09 0.695" rpy="0 0 0" />
         <geometry>
           <box size="0.16 0.02 0.02" />
@@ -276,5 +270,5 @@
       </collision>
       <collision name="base_link_rail_y_3_1">
-        <origin xyz="0.02 0 0.695" rpy="0 0 0" />
+        <origin xyz="-0.05 0 0.695" rpy="0 0 0" />
         <geometry>
           <box size="0.02 0.16 0.02" />
@@ -282,5 +276,5 @@
       </collision>
       <collision name="base_link_floor_3_center">
-        <origin xyz="-0.07 0 0.7065" rpy="0 0 0" />
+        <origin xyz="-0.14 0 0.7065" rpy="0 0 0" />
         <geometry>
           <box size="0.16 0.2 0.003" />
@@ -288,5 +282,5 @@
       </collision>
       <collision name="base_link_floor_3_end_-1">
-        <origin xyz="-0.16 0 0.7065" rpy="0 0 0" />
+        <origin xyz="-0.23 0 0.7065" rpy="0 0 0" />
         <geometry>
           <box size="0.02 0.16 0.003" />
@@ -294,5 +288,5 @@
       </collision>
       <collision name="base_link_floor_3_end_1">
-        <origin xyz="0.02 0 0.7065" rpy="0 0 0" />
+        <origin xyz="-0.05 0 0.7065" rpy="0 0 0" />
         <geometry>
           <box size="0.02 0.16 0.003" />
@@ -300,5 +294,5 @@
       </collision>
       <collision name="base_link_front_door_lower">
-        <origin xyz="0.031 0 0.414" rpy="0 0 0" />
+        <origin xyz="-0.039 0 0.414" rpy="0 0 0" />
         <geometry>
           <box size="0.002 0.2 0.378" />
@@ -306,5 +300,5 @@
       </collision>
       <collision name="base_link_front_door_upper">
-        <origin xyz="0.031 0 0.67375" rpy="0 0 0" />
+        <origin xyz="-0.039 0 0.67375" rpy="0 0 0" />
         <geometry>
           <box size="0.002 0.2 0.0225" />
@@ -312,5 +306,5 @@
       </collision>
       <collision name="base_link_front_door_left_strip">
-        <origin xyz="0.031 0.089 0.63275" rpy="0 0 0" />
+        <origin xyz="-0.039 0.089 0.63275" rpy="0 0 0" />
         <geometry>
           <box size="0.002 0.022 0.0595" />
@@ -318,5 +312,5 @@
       </collision>
       <collision name="base_link_front_door_right_strip">
-        <origin xyz="0.031 -0.089 0.63275" rpy="0 0 0" />
+        <origin xyz="-0.039 -0.089 0.63275" rpy="0 0 0" />
         <geometry>
           <box size="0.002 0.022 0.0595" />
@@ -324,5 +318,5 @@
       </collision>
       <collision name="base_link_rear_door_closed">
-        <origin xyz="-0.171 0 0.455" rpy="0 0 0" />
+        <origin xyz="-0.241 0 0.455" rpy="0 0 0" />
         <geometry>
           <box size="0.002 0.2 0.46" />
@@ -330,5 +324,5 @@
       </collision>
       <collision name="base_link_side_-1_lower">
-        <origin xyz="-0.07 -0.101 0.3575" rpy="0 0 0" />
+        <origin xyz="-0.14 -0.101 0.3575" rpy="0 0 0" />
         <geometry>
           <box size="0.2 0.002 0.265" />
@@ -336,5 +330,5 @@
       </collision>
       <collision name="base_link_side_-1_upper">
-        <origin xyz="-0.07 -0.101 0.6425" rpy="0 0 0" />
+        <origin xyz="-0.14 -0.101 0.6425" rpy="0 0 0" />
         <geometry>
           <box size="0.2 0.002 0.085" />
@@ -342,5 +336,5 @@
       </collision>
       <collision name="base_link_side_-1_front_strip">
-        <origin xyz="0.0075 -0.101 0.545" rpy="0 0 0" />
+        <origin xyz="-0.0625 -0.101 0.545" rpy="0 0 0" />
         <geometry>
           <box size="0.045 0.002 0.11" />
@@ -348,5 +342,5 @@
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
File: underbot_description/urdf/sensors.xacro (robot description, xacro)
@@ -32,5 +32,5 @@
         </geometry>
         <material name="matte_black">
-          <color rgba="0.045 0.05 0.055 1" />
+          <color rgba="0.008 0.009 0.011 1" />
         </material>
       </visual>
@@ -99,5 +99,5 @@
       <parent link="base_link" />
       <child link="camera_mount" />
-      <origin xyz="-0.005 0 0.635" rpy="0 0 0" />
+      <origin xyz="-0.075 0 0.635" rpy="0 0 0" />
     </joint>
     <joint name="camera_optical_joint" type="fixed">
@@ -109,5 +109,5 @@
       <parent link="base_link" />
       <child link="lidar_mount" />
-      <origin xyz="-0.07 0 0.733" rpy="0 0 0" />
+      <origin xyz="-0.14 0 0.733" rpy="0 0 0" />
     </joint>
     <joint name="lidar_scan_joint" type="fixed">

File: underbot_description/urdf/underbot.gazebo.urdf (robot description, URDF)
Before this commit: robot underbot, 23 links, 22 joints
Links:
- link base_link: mass 14.8710078 -> 14.7872478; geometry collision box size=0.002 0.022 0.0595; collision box size=0.002 0.022 0.0595
- link caster_link: geometry collision cylinder length=0.055 radius=0.0395; visual mesh filename=../meshes/caster_link.stl scale=1 1 1
- link left_wheel: geometry collision cylinder length=0.04 radius=0.1025; visual mesh filename=../meshes/left_wheel.stl scale=1 1 1
- link right_wheel: geometry collision cylinder length=0.04 radius=0.1025; visual mesh filename=../meshes/right_wheel.stl scale=1 1 1
Joints:
- joint camera_mount_joint: origin xyz=-0.005 0 0.635 rpy=0 0 0 -> xyz=-0.075 0 0.635 rpy=0 0 0
- joint caster_swivel_joint: origin xyz=0.215 0 0.11 rpy=0 0 0 -> xyz=0.19 0 0.11 rpy=0 0 0
- joint caster_wheel_joint: origin xyz=-0.02 0 -0.07 rpy=0 0 0 -> xyz=-0.02 0 -0.0705 rpy=0 0 0
- joint left_arm_base_joint: origin xyz=-0.07 0.108 0.545 rpy=0 -1.57079632679 -1.57079632679 -> xyz=-0.14 0.108 0.545 rpy=0 -1.57079632679 -1.57079632679
- joint left_wheel_joint: origin xyz=-0.18 0.177 0.0925 rpy=0 0 0 -> xyz=-0.17 0.167 0.1025 rpy=0 0 0
- joint lidar_mount_joint: origin xyz=-0.07 0 0.733 rpy=0 0 0 -> xyz=-0.14 0 0.733 rpy=0 0 0
- joint right_arm_base_joint: origin xyz=-0.07 -0.108 0.545 rpy=0 -1.57079632679 1.57079632679 -> xyz=-0.14 -0.108 0.545 rpy=0 -1.57079632679 1.57079632679
- joint right_wheel_joint: origin xyz=-0.18 -0.177 0.0925 rpy=0 0 0 -> xyz=-0.17 -0.167 0.1025 rpy=0 0 0

File: underbot_description/urdf/underbot.portable.urdf (robot description, URDF)
Before this commit: robot underbot, 23 links, 22 joints
Links:
- link base_link: mass 14.8710078 -> 14.7872478; geometry collision box size=0.002 0.022 0.0595; collision box size=0.002 0.022 0.0595
- link caster_link: geometry collision cylinder length=0.055 radius=0.0395; visual mesh filename=../meshes/caster_link.stl scale=1 1 1
- link left_wheel: geometry collision cylinder length=0.04 radius=0.1025; visual mesh filename=../meshes/left_wheel.stl scale=1 1 1
- link right_wheel: geometry collision cylinder length=0.04 radius=0.1025; visual mesh filename=../meshes/right_wheel.stl scale=1 1 1
Joints:
- joint camera_mount_joint: origin xyz=-0.005 0 0.635 rpy=0 0 0 -> xyz=-0.075 0 0.635 rpy=0 0 0
- joint caster_swivel_joint: origin xyz=0.215 0 0.11 rpy=0 0 0 -> xyz=0.19 0 0.11 rpy=0 0 0
- joint caster_wheel_joint: origin xyz=-0.02 0 -0.07 rpy=0 0 0 -> xyz=-0.02 0 -0.0705 rpy=0 0 0
- joint left_arm_base_joint: origin xyz=-0.07 0.108 0.545 rpy=0 -1.57079632679 -1.57079632679 -> xyz=-0.14 0.108 0.545 rpy=0 -1.57079632679 -1.57079632679
- joint left_wheel_joint: origin xyz=-0.18 0.177 0.0925 rpy=0 0 0 -> xyz=-0.17 0.167 0.1025 rpy=0 0 0
- joint lidar_mount_joint: origin xyz=-0.07 0 0.733 rpy=0 0 0 -> xyz=-0.14 0 0.733 rpy=0 0 0
- joint right_arm_base_joint: origin xyz=-0.07 -0.108 0.545 rpy=0 -1.57079632679 1.57079632679 -> xyz=-0.14 -0.108 0.545 rpy=0 -1.57079632679 1.57079632679
- joint right_wheel_joint: origin xyz=-0.18 -0.177 0.0925 rpy=0 0 0 -> xyz=-0.17 -0.167 0.1025 rpy=0 0 0

File: underbot_description/urdf/underbot.textured.urdf (robot description, URDF)
Before this commit: robot underbot, 23 links, 22 joints
Links:
- link base_link: mass 14.8710078 -> 14.7872478; geometry collision box size=0.002 0.022 0.0595; collision box size=0.002 0.022 0.0595
- link caster_link: geometry collision cylinder length=0.055 radius=0.0395; visual mesh filename=../meshes/caster_link.obj scale=1 1 1
- link left_wheel: geometry collision cylinder length=0.04 radius=0.1025; visual mesh filename=../meshes/left_wheel.obj scale=1 1 1
- link right_wheel: geometry collision cylinder length=0.04 radius=0.1025; visual mesh filename=../meshes/right_wheel.obj scale=1 1 1
Joints:
- joint camera_mount_joint: origin xyz=-0.005 0 0.635 rpy=0 0 0 -> xyz=-0.075 0 0.635 rpy=0 0 0
- joint caster_swivel_joint: origin xyz=0.215 0 0.11 rpy=0 0 0 -> xyz=0.19 0 0.11 rpy=0 0 0
- joint caster_wheel_joint: origin xyz=-0.02 0 -0.07 rpy=0 0 0 -> xyz=-0.02 0 -0.0705 rpy=0 0 0
- joint left_arm_base_joint: origin xyz=-0.07 0.108 0.545 rpy=0 -1.57079632679 -1.57079632679 -> xyz=-0.14 0.108 0.545 rpy=0 -1.57079632679 -1.57079632679
- joint left_wheel_joint: origin xyz=-0.18 0.177 0.0925 rpy=0 0 0 -> xyz=-0.17 0.167 0.1025 rpy=0 0 0
- joint lidar_mount_joint: origin xyz=-0.07 0 0.733 rpy=0 0 0 -> xyz=-0.14 0 0.733 rpy=0 0 0
- joint right_arm_base_joint: origin xyz=-0.07 -0.108 0.545 rpy=0 -1.57079632679 1.57079632679 -> xyz=-0.14 -0.108 0.545 rpy=0 -1.57079632679 1.57079632679
- joint right_wheel_joint: origin xyz=-0.18 -0.177 0.0925 rpy=0 0 0 -> xyz=-0.17 -0.167 0.1025 rpy=0 0 0
