Commit message: Correct WR141E geometry and four-panel Underbot R10 enclosure

File: underbot_description/urdf/underbot.urdf (robot description, URDF)
Before this commit: robot underbot, 23 links, 22 joints
Links:
- link base_link: mass 14.8710078 -> 14.7872478; geometry collision box size=0.002 0.022 0.0595; collision box size=0.002 0.022 0.0595
- link caster_link: geometry collision cylinder length=0.055 radius=0.0395; visual mesh filename=package://underbot_description/meshes/caster_link.stl scale=1 1 1
- link left_wheel: geometry collision cylinder length=0.04 radius=0.1025; visual mesh filename=package://underbot_description/meshes/left_wheel.stl scale=1 1 1
- link right_wheel: geometry collision cylinder length=0.04 radius=0.1025; visual mesh filename=package://underbot_description/meshes/right_wheel.stl scale=1 1 1
Joints:
- joint camera_mount_joint: origin xyz=-0.005 0 0.635 rpy=0 0 0 -> xyz=-0.075 0 0.635 rpy=0 0 0
- joint caster_swivel_joint: origin xyz=0.215 0 0.11 rpy=0 0 0 -> xyz=0.19 0 0.11 rpy=0 0 0
- joint caster_wheel_joint: origin xyz=-0.02 0 -0.07 rpy=0 0 0 -> xyz=-0.02 0 -0.0705 rpy=0 0 0
- joint left_arm_base_joint: origin xyz=-0.07 0.108 0.545 rpy=0 -1.57079632679 -1.57079632679 -> xyz=-0.14 0.108 0.545 rpy=0 -1.57079632679 -1.57079632679
- joint left_wheel_joint: origin xyz=-0.18 0.177 0.0925 rpy=0 0 0 -> xyz=-0.17 0.167 0.1025 rpy=0 0 0
- joint lidar_mount_joint: origin xyz=-0.07 0 0.733 rpy=0 0 0 -> xyz=-0.14 0 0.733 rpy=0 0 0
- joint right_arm_base_joint: origin xyz=-0.07 -0.108 0.545 rpy=0 -1.57079632679 1.57079632679 -> xyz=-0.14 -0.108 0.545 rpy=0 -1.57079632679 1.57079632679
- joint right_wheel_joint: origin xyz=-0.18 -0.177 0.0925 rpy=0 0 0 -> xyz=-0.17 -0.167 0.1025 rpy=0 0 0

File: underbot_description/validation/xacro_expanded.urdf (robot description, URDF)
Before this commit: robot underbot, 23 links, 22 joints
Links:
- link base_link: mass 14.8710078 -> 14.7872478; geometry collision box size=0.002 0.022 0.0595; collision box size=0.002 0.022 0.0595
- link caster_link: geometry collision cylinder length=0.055 radius=0.0395; visual mesh filename=package://underbot_description/meshes/caster_link.stl scale=1 1 1
- link left_wheel: geometry collision cylinder length=0.04 radius=0.1025; visual mesh filename=package://underbot_description/meshes/left_wheel.stl scale=1 1 1
- link right_wheel: geometry collision cylinder length=0.04 radius=0.1025; visual mesh filename=package://underbot_description/meshes/right_wheel.stl scale=1 1 1
Joints:
- joint camera_mount_joint: origin xyz=-0.005 0 0.635 rpy=0 0 0 -> xyz=-0.075 0 0.635 rpy=0 0 0
- joint caster_swivel_joint: origin xyz=0.215 0 0.11 rpy=0 0 0 -> xyz=0.19 0 0.11 rpy=0 0 0
- joint caster_wheel_joint: origin xyz=-0.02 0 -0.07 rpy=0 0 0 -> xyz=-0.02 0 -0.0705 rpy=0 0 0
- joint left_arm_base_joint: origin xyz=-0.07 0.108 0.545 rpy=0 -1.57079632679 -1.57079632679 -> xyz=-0.14 0.108 0.545 rpy=0 -1.57079632679 -1.57079632679
- joint left_wheel_joint: origin xyz=-0.18 0.177 0.0925 rpy=0 0 0 -> xyz=-0.17 0.167 0.1025 rpy=0 0 0
- joint lidar_mount_joint: origin xyz=-0.07 0 0.733 rpy=0 0 0 -> xyz=-0.14 0 0.733 rpy=0 0 0
- joint right_arm_base_joint: origin xyz=-0.07 -0.108 0.545 rpy=0 -1.57079632679 1.57079632679 -> xyz=-0.14 -0.108 0.545 rpy=0 -1.57079632679 1.57079632679
- joint right_wheel_joint: origin xyz=-0.18 -0.177 0.0925 rpy=0 0 0 -> xyz=-0.17 -0.167 0.1025 rpy=0 0 0

File: underbot_flat.urdf (robot description, URDF)
Before this commit: robot underbot, 23 links, 22 joints
Links:
- link base_link: mass 14.8710078 -> 14.7872478; geometry collision box size=0.002 0.022 0.0595; collision box size=0.002 0.022 0.0595
- link caster_link: geometry collision cylinder length=0.055 radius=0.0395; visual mesh filename=underbot_description/meshes/caster_link.stl scale=1 1 1
- link left_wheel: geometry collision cylinder length=0.04 radius=0.1025; visual mesh filename=underbot_description/meshes/left_wheel.stl scale=1 1 1
- link right_wheel: geometry collision cylinder length=0.04 radius=0.1025; visual mesh filename=underbot_description/meshes/right_wheel.stl scale=1 1 1
Joints:
- joint camera_mount_joint: origin xyz=-0.005 0 0.635 rpy=0 0 0 -> xyz=-0.075 0 0.635 rpy=0 0 0
- joint caster_swivel_joint: origin xyz=0.215 0 0.11 rpy=0 0 0 -> xyz=0.19 0 0.11 rpy=0 0 0
- joint caster_wheel_joint: origin xyz=-0.02 0 -0.07 rpy=0 0 0 -> xyz=-0.02 0 -0.0705 rpy=0 0 0
- joint left_arm_base_joint: origin xyz=-0.07 0.108 0.545 rpy=0 -1.57079632679 -1.57079632679 -> xyz=-0.14 0.108 0.545 rpy=0 -1.57079632679 -1.57079632679
- joint left_wheel_joint: origin xyz=-0.18 0.177 0.0925 rpy=0 0 0 -> xyz=-0.17 0.167 0.1025 rpy=0 0 0
- joint lidar_mount_joint: origin xyz=-0.07 0 0.733 rpy=0 0 0 -> xyz=-0.14 0 0.733 rpy=0 0 0
- joint right_arm_base_joint: origin xyz=-0.07 -0.108 0.545 rpy=0 -1.57079632679 1.57079632679 -> xyz=-0.14 -0.108 0.545 rpy=0 -1.57079632679 1.57079632679
- joint right_wheel_joint: origin xyz=-0.18 -0.177 0.0925 rpy=0 0 0 -> xyz=-0.17 -0.167 0.1025 rpy=0 0 0
